File: test.kicad_pcb (KiCad board)
At the start: 2 copper layers, 13.4 x 4.5 mm, 60 parts, among them J1 USB_C_Receptacle_USB2.0_16P, J2 Conn_01x02_Pin (switch), J3 Conn_01x02_Pin (battery), J4 Conn_01x03_Pin, SW1 SW_Push, SW10 SW_Push, SW11 SW_Push, SW12 SW_Push, SW13 SW_Push, SW14 SW_Push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

Commit message: feat(pcb): upgrade it
Parts:
- C1, C10, C2, C3, C4, C5, C6, C7, C8, C9: footprint Capacitor_SMD:C_0201_0603Metric -> Capacitor_SMD:C_0805_2012Metric_Pad1.18x1.45mm_HandSolder
- D19: footprint LED_SMD:LED_PLCC-2_3.4x3.0mm_AK -> LED_SMD:LED_0201_0603Metric_Pad0.64x0.40mm_HandSolder
- R2, R3, R5, R6: footprint Resistor_SMD:R_0201_0603Metric -> Resistor_SMD:R_0805_2012Metric_Pad1.20x1.40mm_HandSolder
- moved D5 159.7 mm to (184.9, 64.8), turned to 180 degrees
- moved D10 159.2 mm to (185.0, 83.5), turned to 180 degrees
- moved D15 158.4 mm to (185.1, 102.2), turned to 180 degrees
- moved D4 138.3 mm to (184.9, 68.5), turned to 180 degrees
- moved D9 136.5 mm to (185.0, 87.2), turned to 180 degrees
- moved D14 135.0 mm to (185.1, 106.0), turned to 180 degrees
- moved D3 117.7 mm to (185.0, 72.2), turned to 180 degrees
- moved D8 115.0 mm to (185.0, 91.0), turned to 180 degrees
- moved D13 113.2 mm to (185.1, 109.8), turned to 180 degrees
- moved D18 112.9 mm to (185.1, 121.0), turned to 180 degrees
- moved D2 97.6 mm to (185.0, 76.0), turned to 180 degrees
- moved D7 93.8 mm to (184.9, 94.8), turned to 180 degrees
- moved D12 91.2 mm to (185.1, 113.5), turned to 180 degrees
- moved D17 89.8 mm to (185.0, 124.8), turned to 180 degrees
- moved SW5 88.9 mm to (102.0, 71.0), turned to 180 degrees
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Routing:
- net row_2: track 182.2 -> 34.1 mm
- net row_1: track 171.6 -> 25.7 mm
- net row_3: track 186.6 -> 51.7 mm
- net col_5: track 250.2 -> 150.1 mm
- net row_4: track 161.4 -> 61.4 mm
- net col_3: track 225.8 -> 128.0 mm
- net col_2: track 201.2 -> 108.1 mm
- net col_4: track 222.5 -> 130.3 mm
- net col_1: track 172.7 -> 88.5 mm
- net Net-(D5-A): track 19.1 -> 86.9 mm
- net Net-(D15-A): track 18.9 -> 86.3 mm
- net Net-(D10-A): track 18.9 -> 86.3 mm
- net Net-(D9-A): track 19.1 -> 81.6 mm
- net D- (post-ESD): track 71.1 -> 13.2 mm, vias 0 -> 2
- net Net-(D14-A): track 18.9 -> 69.2 mm
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- added copper zone on F.Cu, net GND
Other:
- board size 13.4 x 4.5 mm -> 139.2 x 72.4 mm
