File: test.kicad_sch (KiCad schematic)
At the start: 36 parts, among them SW1 SW_Push, SW10 SW_Push, SW11 SW_Push, SW12 SW_Push, SW13 SW_Push, SW14 SW_Push, SW15 SW_Push, SW16 SW_Push, SW17 SW_Push, SW18 SW_Push, SW2 SW_Push, SW3 SW_Push, SW4 SW_Push, SW5 SW_Push, SW6 SW_Push, SW7 SW_Push, SW8 SW_Push, SW9 SW_Push

Commit message: feat: add flake
Parts:
- added C1, C10, C3, C8: C (100nF), Capacitor_SMD:C_0201_0603Metric, symbol Device:C
- added C2: C (10µF), Capacitor_SMD:C_0201_0603Metric, symbol Device:C
- added C4, C5, C9: C (4.7µF), Capacitor_SMD:C_0201_0603Metric, symbol Device:C
- added C6, C7: C (1µF), Capacitor_SMD:C_0201_0603Metric, symbol Device:C
- added D19: LED, LED_SMD:LED_PLCC-2_3.4x3.0mm_AK, symbol Device:LED
- added J1: USB_C_Receptacle_USB2.0_16P, Connector_USB:USB_C_Receptacle_Amphenol_12401948E412A, symbol Connector:USB_C_Receptacle_USB2.0_16P
- added J2: Conn_01x02_Pin (switch), Connector_JST:JST_SH_SM02B-SRSS-TB_1x02-1MP_P1.00mm_Horizontal, symbol Connector:Conn_01x02_Pin
- added J3: Conn_01x02_Pin (battery), Connector_JST:JST_SH_SM02B-SRSS-TB_1x02-1MP_P1.00mm_Horizontal, symbol Connector:Conn_01x02_Pin
- added J4: Conn_01x03_Pin, Connector_JST:JST_SH_SM03B-SRSS-TB_1x03-1MP_P1.00mm_Horizontal, symbol Connector:Conn_01x03_Pin
- added R2: R (470), Resistor_SMD:R_0201_0603Metric, symbol Device:R
- added R3: R (5k), Resistor_SMD:R_0201_0603Metric, symbol Device:R
- added R5, R6: R (5.1k), Resistor_SMD:R_0201_0603Metric, symbol Device:R
- added SW19: SW_Push, Button_Switch_SMD:SW_Push_SPST_NO_Alps_SKRK, symbol Switch:SW_Push
- added U1: E73-2G4M08S1C, E73-2G4M08S1C:E73-2G4M08S1C, symbol E73-2G4M08S1C:E73-2G4M08S1C
- added U2: AP2112K-3.3, Package_TO_SOT_SMD:SOT-23-5, symbol Regulator_Linear:AP2112K-3.3
- added U3: MCP73831-2-OT, Package_TO_SOT_SMD:SOT-23-5, symbol Battery_Management:MCP73831-2-OT
- added U4: USBLC6-2SC6, Package_TO_SOT_SMD:SOT-23-6, symbol Power_Protection:USBLC6-2SC6
Connections:
- net col_1: now also U1.32 (P0.20)
- net col_2: now also U1.30 (P0.17)
- net col_3: now also U1.28 (P0.15)
- net col_4: now also U1.12 (P0.26)
- net col_5: now also U1.14 (P0.06)
- net row_1: now also U1.16 (P0.08)
- net row_2: now also U1.18 (P0.04/AIN2)
- net row_3: now also U1.20 (P0.12)
- net row_4: now also U1.22 (P0.07)
- new net: D19.2 (A), R2.1
- new net: D19.1 (K), U3.1 (STAT)
- new net: R3.2, U3.5 (PROG)
- new net: J1.A5 (CC1), R5.2
- new net: C1.1, SW19.2
- new net: C8.2, C9.1
- new net: C1.2, U1.26 (P0.18/RESET)
- new net: J1.B5 (CC2), R6.2
- new net: J2.1 (Pin_1), J3.2 (Pin_2)
- new net 3v3: C10.2, C7.1, C8.1, U1.19 (VDD), U1.23 (VDDH), U2.5 (VOUT)
- new net BAT: C5.1, J2.2 (Pin_2), U3.3 (V_{BAT})
- new net D+ (post-ESD): U1.31 (D+), U4.6 (I/O1)
- new net D+ (pre-ESD): J1.A6 (D+), J1.B6 (D+), U4.1 (I/O1)
- new net D- (post-ESD): U1.29 (D-), U4.4 (I/O2)
- new net D- (pre-ESD): J1.A7 (D-), J1.B7 (D-), U4.2 (GND)
- new net GND: C10.1, C2.1, C3.1, C4.1, C5.2, C6.1, C7.2, C9.2, J1.A1 (GND), J1.A12 (GND), J1.B1 (GND), J1.B12 (GND), J1.SH (SHIELD), J3.1 (Pin_1), J4.2 (Pin_2), R3.1, R5.1, R6.1, SW19.1, U1.21 (GND), U1.24 (GND), U1.5 (GND), U2.2 (GND), U3.2 (V_{SS}), U4.3 (I/O2)
- new net SWDCLK: J4.1 (Pin_1), U1.39 (SWDCLK)
- new net SWDIO: J4.3 (Pin_3), U1.37 (SWDIO)
- new net VBUS: C2.2, C3.2, C4.2, J1.A4 (VBUS), J1.A9 (VBUS), J1.B4 (VBUS), J1.B9 (VBUS), R2.2, U1.27 (VBUS), U3.4 (V_{DD}), U4.5 (VBUS)
- new net VSYS: C6.2, U2.1 (VIN), U2.3 (EN)
- no-connect marks 0 -> 25
Other:
- note added: "Battery Logic"
- note added: "Charger"
- note added: "Chip"
- note added: "E73-2G4M08S1C"
- note added: "ESD between connector and MCU"
- note added: "LDO"
- note added: "Raspberry Pi Debug Probe (SWD)"
- note added: "USB-C Connector"
- moved on the sheet: D1, D10, D11, D12, D13, D14, D15, D16, D17, D18, D2, D3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

Commit message: feat: init pcb
Connections:
- net 3v3: no longer C8.1, U1.19 (VDD)
- net col_1: now also U1.10 (P0.30/AIN6*); no longer U1.32 (P0.20)
- net col_2: now also U1.9 (P0.31/AIN7*); no longer U1.30 (P0.17)
- net col_3: now also U1.8 (P0.29/AIN5*); no longer U1.28 (P0.15)
- net col_4: now also U1.7 (P0.02/AIN0*); no longer U1.12 (P0.26)
- net col_5: now also U1.6 (P1.13*); no longer U1.14 (P0.06)
- net row_1: now also U1.11 (P0.00/XL1); no longer U1.16 (P0.08)
- net row_2: now also U1.13 (P0.01/XL2); no longer U1.18 (P0.04/AIN2)
- net row_3: now also U1.15 (P0.05/AIN3); no longer U1.20 (P0.12)
- net row_4: now also U1.17 (P1.09); no longer U1.22 (P0.07)
- new net: C8.1, U1.19 (VDD)
Other:
- moved on the sheet: C1, C10, C4, C5, C6, C7, C8, C9, D19, J4, R2, R3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

Commit message: feat(pcb): upgrade it
Parts:
- C1, C10, C2, C3, C4, C5, C6, C7, C8, C9: footprint Capacitor_SMD:C_0201_0603Metric -> Capacitor_SMD:C_0805_2012Metric_Pad1.18x1.45mm_HandSolder
- D19: footprint LED_SMD:LED_PLCC-2_3.4x3.0mm_AK -> LED_SMD:LED_0201_0603Metric_Pad0.64x0.40mm_HandSolder
- R2, R3, R5, R6: footprint Resistor_SMD:R_0201_0603Metric -> Resistor_SMD:R_0805_2012Metric_Pad1.20x1.40mm_HandSolder
Changed lines of the file:
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@@
 			)
 		)
-		(property "Footprint" "Capacitor_SMD:C_0201_0603Metric"
+		(property "Footprint" "Capacitor_SMD:C_0805_2012Metric_Pad1.18x1.45mm_HandSolder"
 			(at 53.0352 148.59 0)
 			(hide yes)
@@
 			)
 		)
-		(property "Footprint" "Resistor_SMD:R_0201_0603Metric"
+		(property "Footprint" "Resistor_SMD:R_0805_2012Metric_Pad1.20x1.40mm_HandSolder"
 			(at 140.208 83.82 90)
 			(hide yes)
@@
 			)
 		)
-		(property "Footprint" "Resistor_SMD:R_0201_0603Metric"
+		(property "Footprint" "Resistor_SMD:R_0805_2012Metric_Pad1.20x1.40mm_HandSolder"
 			(at 137.668 125.73 90)
 			(hide yes)
@@
 			)
 		)
-		(property "Footprint" "Capacitor_SMD:C_0201_0603Metric"
+		(property "Footprint" "Capacitor_SMD:C_0805_2012Metric_Pad1.18x1.45mm_HandSolder"
 			(at 261.3152 96.52 0)
 			(hide yes)
@@
 			)
 		)
-		(property "Footprint" "Resistor_SMD:R_0201_0603Metric"
+		(property "Footprint" "Resistor_SMD:R_0805_2012Metric_Pad1.20x1.40mm_HandSolder"
 			(at 65.278 182.88 90)
 			(hide yes)
@@
 			)
 		)
-		(property "Footprint" "Capacitor_SMD:C_0201_0603Metric"
+		(property "Footprint" "Capacitor_SMD:C_0805_2012Metric_Pad1.18x1.45mm_HandSolder"
 			(at 142.24 151.4348 0)
 			(hide yes)
@@
 			)
 		)
-		(property "Footprint" "Capacitor_SMD:C_0201_0603Metric"
+		(property "Footprint" "Capacitor_SMD:C_0805_2012Metric_Pad1.18x1.45mm_HandSolder"
 			(at 272.7452 135.89 0)
 			(hide yes)
@@
 			)
 		)
-		(property "Footprint" "Capacitor_SMD:C_0201_0603Metric"
+		(property "Footprint" "Capacitor_SMD:C_0805_2012Metric_Pad1.18x1.45mm_HandSolder"
 			(at 113.03 151.4348 0)
 			(hide yes)
@@
 			)
 		)
-		(property "Footprint" "Resistor_SMD:R_0201_0603Metric"
+		(property "Footprint" "Resistor_SMD:R_0805_2012Metric_Pad1.20x1.40mm_HandSolder"
 			(at 52.578 182.88 90)
 			(hide yes)
@@
 			)
 		)
-		(property "Footprint" "Capacitor_SMD:C_0201_0603Metric"
+		(property "Footprint" "Capacitor_SMD:C_0805_2012Metric_Pad1.18x1.45mm_HandSolder"
 			(at 238.4552 46.99 0)
 			(hide yes)
@@
 			)
 		)
-		(property "Footprint" "LED_SMD:LED_PLCC-2_3.4x3.0mm_AK"
+		(property "Footprint" "LED_SMD:LED_0201_0603Metric_Pad0.64x0.40mm_HandSolder"
 			(at 138.43 93.98 0)
 			(hide yes)
@@
 			)
 		)
-		(property "Footprint" "Capacitor_SMD:C_0201_0603Metric"
+		(property "Footprint" "Capacitor_SMD:C_0805_2012Metric_Pad1.18x1.45mm_HandSolder"
 			(at 69.5452 148.59 0)
 			(hide yes)
@@
 			)
 		)
-		(property "Footprint" "Capacitor_SMD:C_0201_0603Metric"
+		(property "Footprint" "Capacitor_SMD:C_0805_2012Metric_Pad1.18x1.45mm_HandSolder"
 			(at 272.7452 147.32 0)
 			(hide yes)
@@
 			)
 		)
-		(property "Footprint" "Capacitor_SMD:C_0201_0603Metric"
+		(property "Footprint" "Capacitor_SMD:C_0805_2012Metric_Pad1.18x1.45mm_HandSolder"
 			(at 122.2248 76.2 0)
 			(hide yes)
@@
 			)
 		)
-		(property "Footprint" "Capacitor_SMD:C_0201_0603Metric"
+		(property "Footprint" "Capacitor_SMD:C_0805_2012Metric_Pad1.18x1.45mm_HandSolder"
 			(at 118.4148 110.49 0)
 			(hide yes)
